Commit message: ROS2Lab v18 (work in progress): Jazzy-correct controllers and sensors, MoveIt 2 for all arms
- Gazebo worlds no longer download Sun/Ground Plane from Fuel (world failed to load offline)
- one spawner for all controllers (parallel spawners deadlock on Jazzy's spawner lock)
- GZ_SIM_RESOURCE_PATH set by the sim launch files so Gazebo finds the meshes
- MoveIt 2 config packages (SRDF, OMPL/Pilz/CHOMP/STOMP, ros2_control) for the 12 vendor arms
- browser move_group + RViz MotionPlanning panel; xacro.load_yaml support
- simulations for Scout, Spot, Crazyflie and auto-generated ones for robots without a spec
- teleop: holonomic and up/down keys; robots stop at world obstacles

Co-Authored-By: Claude Opus 5.5 <noreply@anthropic.com>
Claude-Session: https://claude.ai/code/session_01RqxNJg8jb98FbU2R3yzkJ8

File: ros2lab-course/public/robots/scout_description/urdf/scout_v2.urdf (robot description, URDF)
Before this commit: robot scout_v2, 7 links, 6 joints
Joints:
- joint front_left_wheel: type fixed -> continuous
- joint front_right_wheel: type fixed -> continuous
- joint rear_left_wheel: type fixed -> continuous
- joint rear_right_wheel: type fixed -> continuous
