Commit message: Fix Magician URDF limits (mimic joints and right jaw) rejected by MoveIt; RViz robot copies with COLLADA material arrays
Co-Authored-By: Claude Opus 5.5 <noreply@anthropic.com>
Claude-Session: https://claude.ai/code/session_01RqxNJg8jb98FbU2R3yzkJ8

File: ros2lab-course/public/robots/dobot_description/urdf/magician.urdf (robot description, URDF)
Before this commit: robot magician, 10 links, 9 joints
Joints:
- joint magician_joint_mimic_1: limit lower=0.0 upper=6.283185307179586 effort=2000 velocity=1 -> lower=-6.283185307179586 upper=6.283185307179586 effort=2000 velocity=1
- joint magician_joint_mimic_2: limit lower=0.0 upper=6.283185307179586 effort=2000 velocity=1 -> lower=-6.283185307179586 upper=6.283185307179586 effort=2000 velocity=1
- joint magician_joint_prismatic_r: limit lower=0 upper=-0.0135 effort=2000 velocity=1 -> lower=-0.0135 upper=0 effort=2000 velocity=1
