Commit message: Crazyflie URDF: add inertia and collision so Gazebo keeps the link (real gz dropped the model)
Co-Authored-By: Claude Opus 5.5 <noreply@anthropic.com>
Claude-Session: https://claude.ai/code/session_01RqxNJg8jb98FbU2R3yzkJ8

File: ros2lab-course/public/robots/crazyflie_description/urdf/crazyflie.urdf (robot description, URDF)
Before this commit: robot cf, 1 links, 0 joints
Links:
- link cf: mass None -> 0.027; geometry collision box size=0.092 0.092 0.029; visual mesh filename=package://crazyflie_description/meshes/urdf/cf2_assembly_wi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 scale=1.0 1.0 1.0
